File: Boards/Controller/DisplayController.brd (EAGLE design)
At the start: 52.9 x 39 mm, 47 parts, among them J1 USB0001LF, J100 38K8067, J3 AVR_SPI_PRG_62X3_LOCK, Q1 BSS138, U1 MCP1703CB, U100 MCP73831, U101 MAX1797, U2 FT232RQ, U3 ATMEGA328P-MU, U5 MAX1704X, X2 CRYSTAL7A-20.000MAAJ-T

Commit message: updated part info
Parts:
- D1: device MyParts:SML1206 -> led:1206
Routing:
- net RESET: track 62.1 -> 59.0 mm
- net VCC: track 127.6 -> 125.7 mm
Other:
- board text added: "Rev. 125"
- board text removed: "Rev. 126"
Changed lines of the file:
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@@
 <rectangle x1="38.8" y1="33.25" x2="52.936" y2="39" layer="41"/>
 <text x="9.6378" y="36.9484" size="1.4" layer="21" font="vector" ratio="13" rot="SR0">3216 Bluetooth Controller </text>
-<text x="0.4826" y="7.2644" size="1.016" layer="21" font="vector" ratio="12" rot="SR270">Rev. 126</text>
+<text x="0.4826" y="7.2644" size="1.016" layer="21" font="vector" ratio="12" rot="SR270">Rev. 125</text>
 </plain>
 <attributes>
@@
 <element name="C13" library="SparkFun" package="0603-CAP" value="100nF" x="17.5768" y="32.766"/>
 <element name="S3" library="SparkFun" package="TACTILE_SWITCH_SMD" value="SWITCH-MOMENTARY-2SMD" x="33.5786" y="29.4332" rot="R270"/>
-<element name="D1" library="MyParts" package="SML1206" value="" x="33.5786" y="35.5852">
+<element name="D1" library="led" package="1206" value="" x="33.5786" y="35.5852">
 <attribute name="NEWARK_PN" value="09J8040" x="33.5786" y="35.5852" size="1.778" layer="27" display="off"/>
 </element>
@@
 <wire x1="32.7914" y1="32.9442" x2="33.3752" y2="33.528" width="0.254" layer="1"/>
 <wire x1="33.3752" y1="33.528" x2="34.5948" y2="33.528" width="0.254" layer="1"/>
-<wire x1="31.8286" y1="35.5852" x2="35.0006" y2="33.9338" width="0.254" layer="1"/>
+<wire x1="35.0006" y1="35.5852" x2="35.0006" y2="33.9338" width="0.254" layer="1"/>
 <wire x1="35.0006" y1="33.9338" x2="34.5948" y2="33.528" width="0.254" layer="1"/>
 </signal>
@@
 <wire x1="31.6736" y1="35.6364" x2="31.75" y2="35.56" width="0.254" layer="1"/>
 <wire x1="31.75" y1="35.56" x2="32.1314" y2="35.56" width="0.254" layer="1"/>
-<wire x1="32.1314" y1="35.56" x2="35.3286" y2="35.5852" width="0.254" layer="1"/>
+<wire x1="32.1314" y1="35.56" x2="32.1566" y2="35.5852" width="0.254" layer="1"/>
 </signal>
 <signal name="N$5">
